File: A2600 Keyboard/A2600 Keyboard.sch (KiCad schematic (older format))
At the start: 15 parts, among them J1 Atari_IDC, SW1 1, SW10 *, SW11 0, SW12 #, SW2 2, SW3 3, SW4 4, SW5 5, SW6 6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

Commit message: Layout done
Parts:
- added M1, M2, M3, M4: Mounting, mounting:M3_pin, symbol mounting:Mounting
- J1: footprint (none) -> IDC_Joystick:IDC_Joystick
- R301, R302: footprint (none) -> Resistor_THT:R_Axial_DIN0207_L6.3mm_D2.5mm_P10.16mm_Horizontal
- SW1, SW10, SW11, SW12, SW2, SW3, SW4, SW5, SW6, SW7, SW8, SW9: footprint (none) -> switch_cutout:SW_PUSH_6mm
Changed lines of the file:
@@
 F 0 "J1" H 6012 1815 50  0000 C CNN
 F 1 "Atari_IDC" H 6012 1724 50  0000 C CNN
-F 2 "" H 6025 1075 50  0001 C CNN
+F 2 "IDC_Joystick:IDC_Joystick" H 6025 1075 50  0001 C CNN
 F 3 "" H 6025 1075 50  0001 C CNN
 	1    6000 1400
@@
 F 0 "R302" V 4818 1275 50  0000 C CNN
 F 1 "4k7" V 4909 1275 50  0000 C CNN
-F 2 "" V 4955 1275 50  0001 C CNN
+F 2 "Resistor_THT:R_Axial_DIN0207_L6.3mm_D2.5mm_P10.16mm_Horizontal" V 4955 1275 50  0001 C CNN
 F 3 "~" H 5025 1275 50  0001 C CNN
 	1    5025 1275
@@
 F 0 "SW1" V 6429 2544 50  0000 L CNN
 F 1 "1" V 6520 2544 50  0000 L CNN
-F 2 "" H 6475 2400 50  0001 C CNN
+F 2 "switch_cutout:SW_PUSH_6mm" H 6475 2400 50  0001 C CNN
 F 3 "~" H 6475 2400 50  0001 C CNN
 	1    6475 2400
@@
 F 0 "SW2" V 5854 2544 50  0000 L CNN
 F 1 "2" V 5945 2544 50  0000 L CNN
-F 2 "" H 5900 2400 50  0001 C CNN
+F 2 "switch_cutout:SW_PUSH_6mm" H 5900 2400 50  0001 C CNN
 F 3 "~" H 5900 2400 50  0001 C CNN
 	1    5900 2400
@@
 F 0 "SW3" V 5304 2544 50  0000 L CNN
 F 1 "3" V 5395 2544 50  0000 L CNN
-F 2 "" H 5350 2400 50  0001 C CNN
+F 2 "switch_cutout:SW_PUSH_6mm" H 5350 2400 50  0001 C CNN
 F 3 "~" H 5350 2400 50  0001 C CNN
 	1    5350 2400
@@
 F 0 "SW4" V 6429 3044 50  0000 L CNN
 F 1 "4" V 6520 3044 50  0000 L CNN
-F 2 "" H 6475 2900 50  0001 C CNN
+F 2 "switch_cutout:SW_PUSH_6mm" H 6475 2900 50  0001 C CNN
 F 3 "~" H 6475 2900 50  0001 C CNN
 	1    6475 2900
@@
 F 0 "SW5" V 5854 3044 50  0000 L CNN
 F 1 "5" V 5945 3044 50  0000 L CNN
-F 2 "" H 5900 2900 50  0001 C CNN
+F 2 "switch_cutout:SW_PUSH_6mm" H 5900 2900 50  0001 C CNN
 F 3 "~" H 5900 2900 50  0001 C CNN
 	1    5900 2900
@@
 F 0 "SW6" V 5304 3044 50  0000 L CNN
 F 1 "6" V 5395 3044 50  0000 L CNN
-F 2 "" H 5350 2900 50  0001 C CNN
+F 2 "switch_cutout:SW_PUSH_6mm" H 5350 2900 50  0001 C CNN
 F 3 "~" H 5350 2900 50  0001 C CNN
 	1    5350 2900
@@
 F 0 "SW7" V 6429 3544 50  0000 L CNN
 F 1 "7" V 6520 3544 50  0000 L CNN
-F 2 "" H 6475 3400 50  0001 C CNN
+F 2 "switch_cutout:SW_PUSH_6mm" H 6475 3400 50  0001 C CNN
 F 3 "~" H 6475 3400 50  0001 C CNN
 	1    6475 3400
@@
 F 0 "SW8" V 5854 3544 50  0000 L CNN
 F 1 "8" V 5945 3544 50  0000 L CNN
-F 2 "" H 5900 3400 50  0001 C CNN
+F 2 "switch_cutout:SW_PUSH_6mm" H 5900 3400 50  0001 C CNN
 F 3 "~" H 5900 3400 50  0001 C CNN
 	1    5900 3400
@@
 F 0 "SW9" V 5304 3544 50  0000 L CNN
 F 1 "9" V 5395 3544 50  0000 L CNN
-F 2 "" H 5350 3400 50  0001 C CNN
+F 2 "switch_cutout:SW_PUSH_6mm" H 5350 3400 50  0001 C CNN
 F 3 "~" H 5350 3400 50  0001 C CNN
 	1    5350 3400
@@
 F 0 "SW10" V 6429 4044 50  0000 L CNN
 F 1 "*" V 6520 4044 50  0000 L CNN
-F 2 "" H 6475 3900 50  0001 C CNN
+F 2 "switch_cutout:SW_PUSH_6mm" H 6475 3900 50  0001 C CNN
 F 3 "~" H 6475 3900 50  0001 C CNN
 	1    6475 3900
@@
 F 0 "SW11" V 5854 4044 50  0000 L CNN
 F 1 "0" V 5945 4044 50  0000 L CNN
-F 2 "" H 5900 3900 50  0001 C CNN
+F 2 "switch_cutout:SW_PUSH_6mm" H 5900 3900 50  0001 C CNN
 F 3 "~" H 5900 3900 50  0001 C CNN
 	1    5900 3900
@@
 F 0 "SW12" V 5304 4044 50  0000 L CNN
 F 1 "#" V 5395 4044 50  0000 L CNN
-F 2 "" H 5350 3900 50  0001 C CNN
+F 2 "switch_cutout:SW_PUSH_6mm" H 5350 3900 50  0001 C CNN
 F 3 "~" H 5350 3900 50  0001 C CNN
 	1    5350 3900
@@
 F 0 "R301" V 6793 1275 50  0000 C CNN
 F 1 "4k7" V 6884 1275 50  0000 C CNN
-F 2 "" V 6930 1275 50  0001 C CNN
+F 2 "Resistor_THT:R_Axial_DIN0207_L6.3mm_D2.5mm_P10.16mm_Horizontal" V 6930 1275 50  0001 C CNN
 F 3 "~" H 7000 1275 50  0001 C CNN
 	1    7000 1275
@@
 	5025 800  5025 875
 Connection ~ 5025 875
+$Comp
+L mounting:Mounting M1
+U 1 1 604667D0
+P 10775 550
+F 0 "M1" H 10775 650 50  0001 C CNN
+F 1 "Mounting" H 10775 475 50  0001 C CNN
+F 2 "mounting:M3_pin" H 10775 550 50  0001 C CNN
+F 3 "~" H 10775 550 50  0001 C CNN
+	1    10775 550
+	1    0    0    -1
+$EndComp
+$Comp
+L mounting:Mounting M2
+U 1 1 60467268
+P 10900 550
+F 0 "M2" H 10900 650 50  0001 C CNN
+F 1 "Mounting" H 10900 475 50  0001 C CNN
+F 2 "mounting:M3_pin" H 10900 550 50  0001 C CNN
+F 3 "~" H 10900 550 50  0001 C CNN
+	1    10900 550
+	1    0    0    -1
+$EndComp
+$Comp
+L mounting:Mounting M3
+U 1 1 604685BE
+P 11025 550
+F 0 "M3" H 11025 650 50  0001 C CNN
+F 1 "Mounting" H 11025 475 50  0001 C CNN
+F 2 "mounting:M3_pin" H 11025 550 50  0001 C CNN
+F 3 "~" H 11025 550 50  0001 C CNN
+	1    11025 550
+	1    0    0    -1
+$EndComp
+$Comp
+L mounting:Mounting M4
+U 1 1 60469A3A
+P 11150 550
+F 0 "M4" H 11150 650 50  0001 C CNN
+F 1 "Mounting" H 11150 475 50  0001 C CNN
+F 2 "mounting:M3_pin" H 11150 550 50  0001 C CNN
+F 3 "~" H 11150 550 50  0001 C CNN
+	1    11150 550
+	1    0    0    -1
+$EndComp
 $EndSCHEMATC
