File: faceplates/A2600 Faceplate/A2600 Faceplate.kicad_pcb (KiCad board)
At the start: 2 copper layers, 61 x 99.7 mm, 17 parts, among them M1 Mounting, M2 Mounting, M3 Mounting, M4 Mounting

Commit message: Added Star Raiders
Parts:
- added G***: LOGO, artwork:sr_title, B.Cu at (152.4, 59.1)
- added G***: LOGO, artwork:sr_no_key, B.Cu at (167.6, 105.4)
- added G***: LOGO, artwork:sr_no_key, B.Cu at (152.4, 105.4)
- added G***: LOGO, artwork:sr_no_key, B.Cu at (137.2, 105.4)
- added G***: LOGO, artwork:sr_no_key, B.Cu at (137.2, 90.2)
- added G***: LOGO, artwork:sr_key, B.Cu at (152.4, 90.2)
- added G***: LOGO, artwork:sr_key, B.Cu at (167.6, 90.2)
- added G***: LOGO, artwork:sr_key, B.Cu at (137.2, 74.9)
- added G***: LOGO, artwork:sr_key, B.Cu at (152.4, 74.9)
- added G***: LOGO, artwork:sr_key, B.Cu at (167.6, 74.9)
- added G***: LOGO, artwork:sr_no_key, B.Cu at (137.2, 120.7)
- added G***: LOGO, artwork:sr_no_key, B.Cu at (152.4, 120.7)
- added G***: LOGO, artwork:sr_no_key, B.Cu at (167.6, 120.7)
Other:
- board text added: "COMPUTER ON/OFF"
- board text added: "FORE VIEW"
- board text added: "GAL MAP"
- board text added: "HYPERWARP"
- board text added: "SHIELDS ON/OFF"
- board text removed: "Atari 2600 Keyboard github.com/tebl"
- board text removed: "Licensed under CERN OHL v1.2"
